File: extras/schematic_atmega328_standalone_8MHz_LCD16x2.sch (EAGLE design)
At the start: 28 parts, among them U2 328P, Y1 32.768kHz, Y2 12MHz

Commit message: AKC6955 Arduino Library
Parts:
- Y1: device SparkFun-Clocks:CRYSTAL-32.768KHZPTH-2X6 -> SparkFun-Clocks:CRYSTAL-32.768kHzPTH-2X6
Changed lines of the file:
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@@
 <part name="GND10" library="supply1" library_urn="urn:adsk.eagle:library:371" deviceset="GND" device=""/>
 <part name="U$1" library="AKC" deviceset="AKC6955" device="AKC6955" package3d_urn="urn:adsk.eagle:package:29581846/1"/>
-<part name="Y1" library="SparkFun-Clocks" library_urn="urn:adsk.eagle:library:511" deviceset="CRYSTAL-32.768KHZ" device="PTH-2X6" package3d_urn="urn:adsk.eagle:package:37514/1" value="32.768kHz"/>
+<part name="Y1" library="SparkFun-Clocks" library_urn="urn:adsk.eagle:library:511" deviceset="CRYSTAL-32.768kHz" device="PTH-2X6" package3d_urn="urn:adsk.eagle:package:37514/1" value="32.768kHz"/>
 <part name="C1" library="SparkFun-Capacitors" library_urn="urn:adsk.eagle:library:510" deviceset="22PF" device="-PTH-2.54MM-200V-5%" package3d_urn="urn:adsk.eagle:package:37435/1" value="22pF"/>
 <part name="C2" library="SparkFun-Capacitors" library_urn="urn:adsk.eagle:library:510" deviceset="22PF" device="-PTH-2.54MM-200V-5%" package3d_urn="urn:adsk.eagle:package:37435/1" value="22pF"/>
